Commit message: zzz Alienware update

File: knolling_box/box_0.urdf (robot description, URDF)
Before this commit: robot 2x2, 1 links, 0 joints
Links:
- link base_link: geometry collision box size=0.022 0.02 0.016; visual box size=0.022 0.02 0.016

File: knolling_box/box_1.urdf (robot description, URDF)
Before this commit: robot 2x2, 1 links, 0 joints
Links:
- link base_link: geometry collision box size=0.025 0.022 0.011; visual box size=0.025 0.022 0.011

File: knolling_box/box_2.urdf (robot description, URDF)
Before this commit: robot 2x2, 1 links, 0 joints
Links:
- link base_link: geometry collision box size=0.018 0.017 0.02; visual box size=0.018 0.017 0.02

File: knolling_box/box_3.urdf (robot description, URDF)
Before this commit: robot 2x2, 1 links, 0 joints
Links:
- link base_link: geometry collision box size=0.034 0.02 0.015; visual box size=0.034 0.02 0.015

File: knolling_box/box_4.urdf (robot description, URDF)
Before this commit: robot 2x2, 1 links, 0 joints
Links:
- link base_link: geometry collision box size=0.02 0.018 0.015; visual box size=0.02 0.018 0.015
