Commit message: Update new object urdf file

File: ASSET/urdf/OpensCAD_generate/urdf_file/charger_1_L0.55_T0.55.urdf (robot description, URDF)
Before this commit: robot charger_1_L0.55_T0.55, 1 links, 0 joints
Links:
- link charger_1_L0.55_T0.55Link: geometry collision mesh filename=generated_stl/charger/charger_1/charger_1_L0.55_T0.55/charg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 scale=0.01 0.01 0.01; visual mesh filename=generated_stl/charger/charger_1/charger_1_L0.55_T0.55/charg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 scale=0.01 0.01 0.01

File: ASSET/urdf/OpensCAD_generate/urdf_file/charger_1_L0.60_T0.60.urdf (robot description, URDF)
Before this commit: robot charger_1_L0.60_T0.60, 1 links, 0 joints
Links:
- link charger_1_L0.60_T0.60Link: geometry collision mesh filename=generated_stl/charger/charger_1/charger_1_L0.60_T0.60/charg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 scale=0.01 0.01 0.01; visual mesh filename=generated_stl/charger/charger_1/charger_1_L0.60_T0.60/charg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 scale=0.01 0.01 0.01

File: ASSET/urdf/OpensCAD_generate/urdf_file/charger_1_L0.65_T0.65.urdf (robot description, URDF)
Before this commit: robot charger_1_L0.65_T0.65, 1 links, 0 joints
Links:
- link charger_1_L0.65_T0.65Link: geometry collision mesh filename=generated_stl/charger/charger_1/charger_1_L0.65_T0.65/charg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 scale=0.01 0.01 0.01; visual mesh filename=generated_stl/charger/charger_1/charger_1_L0.65_T0.65/charg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 scale=0.01 0.01 0.01

File: ASSET/urdf/OpensCAD_generate/urdf_file/charger_1_L0.70_T0.70.urdf (robot description, URDF)
Before this commit: robot charger_1_L0.70_T0.70, 1 links, 0 joints
Links:
- link charger_1_L0.70_T0.70Link: geometry collision mesh filename=generated_stl/charger/charger_1/charger_1_L0.70_T0.70/charg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 scale=0.01 0.01 0.01; visual mesh filename=generated_stl/charger/charger_1/charger_1_L0.70_T0.70/charg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 scale=0.01 0.01 0.01

File: ASSET/urdf/OpensCAD_generate/urdf_file/charger_1_L0.75_T0.75.urdf (robot description, URDF)
Before this commit: robot charger_1_L0.75_T0.75, 1 links, 0 joints
Links:
- link charger_1_L0.75_T0.75Link: geometry collision mesh filename=generated_stl/charger/charger_1/charger_1_L0.75_T0.75/charg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 scale=0.01 0.01 0.01; visual mesh filename=generated_stl/charger/charger_1/charger_1_L0.75_T0.75/charg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 scale=0.01 0.01 0.01

File: ASSET/urdf/OpensCAD_generate/urdf_file/charger_1_L0.80_T0.80.urdf (robot description, URDF)
Before this commit: robot charger_1_L0.80_T0.80, 1 links, 0 joints
Links:
- link charger_1_L0.80_T0.80Link: geometry collision mesh filename=generated_stl/charger/charger_1/charger_1_L0.80_T0.80/charg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 scale=0.01 0.01 0.01; visual mesh filename=generated_stl/charger/charger_1/charger_1_L0.80_T0.80/charg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 scale=0.01 0.01 0.01

File: ASSET/urdf/OpensCAD_generate/urdf_file/charger_1_L0.85_T0.85.urdf (robot description, URDF)
Before this commit: robot charger_1_L0.85_T0.85, 1 links, 0 joints
Links:
- link charger_1_L0.85_T0.85Link: geometry collision mesh filename=generated_stl/charger/charger_1/charger_1_L0.85_T0.85/charg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 scale=0.01 0.01 0.01; visual mesh filename=generated_stl/charger/charger_1/charger_1_L0.85_T0.85/charg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 scale=0.01 0.01 0.01

File: ASSET/urdf/OpensCAD_generate/urdf_file/charger_1_L0.90_T0.90.urdf (robot description, URDF)
Before this commit: robot charger_1_L0.90_T0.90, 1 links, 0 joints
Links:
- link charger_1_L0.90_T0.90Link: geometry collision mesh filename=generated_stl/charger/charger_1/charger_1_L0.90_T0.90/charg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 scale=0.01 0.01 0.01; visual mesh filename=generated_stl/charger/charger_1/charger_1_L0.90_T0.90/charg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 scale=0.01 0.01 0.01

File: ASSET/urdf/OpensCAD_generate/urdf_file/charger_1_L0.95_T0.95.urdf (robot description, URDF)
Before this commit: robot charger_1_L0.95_T0.95, 1 links, 0 joints
Links:
- link charger_1_L0.95_T0.95Link: geometry collision mesh filename=generated_stl/charger/charger_1/charger_1_L0.95_T0.95/charg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 scale=0.01 0.01 0.01; visual mesh filename=generated_stl/charger/charger_1/charger_1_L0.95_T0.95/charg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 scale=0.01 0.01 0.01

File: ASSET/urdf/OpensCAD_generate/urdf_file/charger_1_L1.00_T1.00.urdf (robot description, URDF)
Before this commit: robot charger_1_L1.00_T1.00, 1 links, 0 joints
Links:
- link charger_1_L1.00_T1.00Link: geometry collision mesh filename=generated_stl/charger/charger_1/charger_1_L1.00_T1.00/charg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 scale=0.01 0.01 0.01; visual mesh filename=generated_stl/charger/charger_1/charger_1_L1.00_T1.00/charg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 scale=0.01 0.01 0.01
