Commit message: zzz xps update

File: ASSET/urdf/OpensCAD_generate/urdf_file/screwdriver_1_L0.98_T0.98.urdf (robot description, URDF)
Before this commit: robot screwdriver_1_L0.98_T0.98, 1 links, 0 joints
Links:
- link screwdriver_1_L0.98_T0.98Link: mass 0.0 -> 0.1

File: ASSET/urdf/OpensCAD_generate/urdf_file/screwdriver_2_L0.98_T0.99.urdf (robot description, URDF)
Before this commit: robot screwdriver_2_L0.98_T0.99, 1 links, 0 joints
Links:
- link screwdriver_2_L0.98_T0.99Link: mass 0.0 -> 0.1

File: ASSET/urdf/OpensCAD_generate/urdf_file/screwdriver_2_L1.00_T1.04.urdf (robot description, URDF)
Before this commit: robot screwdriver_2_L1.00_T1.04, 1 links, 0 joints
Links:
- link screwdriver_2_L1.00_T1.04Link: mass 0.0 -> 0.1
